File: palmrest/palmrest.kicad_pcb (KiCad board)
At the start: 2 copper layers, 86 x 48.1 mm, 17 parts, among them J1 MJ-4PP-9, J2 Conn_01x05_Female, J3 Conn_01x05_Female, J4 Conn_01x12_Female, J5 Conn_01x12_Female, SW1 SW_PUSH, SW2 SW_SPDT, U1 ProMicro

Commit message: revenge3
Parts:
- removed BT2: Battery_Cell, mammoth:ch28-2032LF_rev
- removed D2: D, mammoth:D_SOD-323_HandSoldering_rev
- removed the G*** at (175.5, 85.3) (x2)
- removed J5: Conn_01x12_Female, mammoth:PinHeader_1x12_P2.54mm_Vertical
- removed SW2: SW_SPDT, mammoth:SS-12D00G3
- added C2: 22μF, mammoth:CP_Radial_D5.0mm_P2.00mm_P5.00mm_rev, F.Cu at (182.5, 87.6)
- added G***: LOGO, mammoth:icon, F.Cu at (166.6, 96.2)
- added G***: LOGO, mammoth:icon, B.Cu at (166.6, 96.2)
- added L1: 100μH, mammoth:L_Radial_D10.0mm_P5.00mm_Fastron_07M, F.Cu at (126.7, 74.3)
- added U2: XIAO, mammoth:Seeeduino XIAO-MOUDLE14P-2.54-21X17.8MM, B.Cu at (130.8, 79.1)
- added U3: HT7733A, mammoth:HT7733A, F.Cu at (199.0, 67.3)
- BT1: footprint mammoth:ch28-2032LF_rev -> mammoth:bat_case_AAA; moved to F.Cu
- C1: value C -> 47μF; footprint mammoth:C_1206_3216Metric_Pad1.33x1.80mm_HandSolder_rev -> mammoth:CP_Radial_D5.0mm_P2.00mm_P5.00mm_rev; moved to F.Cu
- D1: value D -> D_Schottky; footprint mammoth:D_SOD-323_HandSoldering_rev -> mammoth:D_DO-34_SOD68_P7.62mm_Horizontal; moved to F.Cu
- J2: footprint mammoth:JST_ACH_BM05B-ACHSS-A-GAN-ETF_1x05-1MP_P1.20mm_Vertical -> mammoth:JST_ACH_BM05B-ACHSS-A-GAN-ETF_1x05-1MP_P1.20mm_Vertical_rev
- J3: value Conn_01x05_Female -> Conn_01x10_Female; footprint mammoth:JST_ACH_BM05B-ACHSS-A-GAN-ETF_1x05-1MP_P1.20mm_Vertical -> Connector_PinHeader_2.54mm:PinHeader_2x05_P2.54mm_Vertical; moved to F.Cu
- J4: value Conn_01x12_Female -> Conn_01x05_Female; footprint mammoth:PinHeader_1x12_P2.54mm_Vertical -> Connector_PinHeader_2.54mm:PinHeader_1x05_P2.54mm_Vertical
- SW1: value SW_PUSH -> SW_SPDT; footprint mammoth:ResetSW -> mammoth:SS-12D00G3
- U1: value ProMicro -> XIAO; footprint mammoth:ProMicro_v3 -> mammoth:Seeeduino XIAO-MOUDLE14P-2.54-21X17.8MM
- moved J4 53.2 mm to (174.5, 63.8)
- moved D1 42.8 mm to (174.7, 79.8), turned to 0 degrees
- moved C1 26.1 mm to (170.4, 87.6), turned to 0 degrees
- moved J3 20.8 mm to (158.2, 84.8), turned to 0 degrees
- moved BT1 17.3 mm to (123.2, 60.7), turned to -15 degrees
- moved U1 10.9 mm to (148.6, 79.1), turned to 180 degrees
- moved J2 7.24 mm to (177.8, 69.6)
- moved SW1 2.29 mm to (177.5, 97.3)
- moved R2 1.36 mm to (197.9, 93.4)
- moved R1 1.36 mm to (192.0, 93.4)
Connections:
- C1 pad 1: VCC -> Net-(C1-Pad1)
- D1 pad 1: Net-(D1-Pad1) -> VDD
- D1 pad 2: Net-(BT1-Pad1) -> Net-(D1-Pad2)
- J1 pad A: SDA -> GND
- J1 pad C: GND -> SDA
- J1 pad D: VCC -> VDD
- J2 pad 1: LED -> INT
- J2 pad 3: VCC -> VDD
- J3 pad 1: LED -> d7
- J3 pad 2: SDA -> d3
- J3 pad 3: VCC -> d8
- J3 pad 4: GND -> d2
- J3 pad 5: SCL -> d9
- J4 pad 1: Net-(J4-Pad1) -> INT
- J4 pad 2: GND -> SDA
- J4 pad 3: RST -> VDD
- J4 pad 4: VCC -> GND
- J4 pad 5: Net-(J4-Pad5) -> SCL
- R1 pad 1: VCC -> VDD
- R2 pad 1: VCC -> VDD
- SW1 pad 1: RST -> Net-(C1-Pad1)
- SW1 pad 2: GND -> Net-(BT1-Pad1)
- U1 pad 1: LED -> d0
- U1 pad 10: Net-(J5-Pad3) -> d9
- U1 pad 11: Net-(J5-Pad2) -> d10
- U1 pad 12: Net-(J5-Pad1) -> VDD
- U1 pad 13: Net-(J4-Pad12) -> GND
- U1 pad 14: Net-(J4-Pad11) -> VCC
- U1 pad 2: Net-(J5-Pad11) -> d1
- U1 pad 3: GND -> d2
- U1 pad 4: GND -> d3
- U1 pad 7: Net-(J5-Pad6) -> INT
- U1 pad 8: Net-(J5-Pad5) -> d7
- U1 pad 9: Net-(J5-Pad4) -> d8
Routing:
- net GND: track 57.9 -> 278.8 mm, vias 5 -> 7
- net VDD: track 0.00 -> 209.8 mm
- net RST: track 89.1 -> 0.00 mm
- net d0: track 0.00 -> 85.6 mm
- net INT: track 0.00 -> 82.4 mm, vias 0 -> 1
- net SDA: track 111.1 -> 192.5 mm, vias 2 -> 0
- net Net-(D1-Pad2): track 0.00 -> 80.1 mm
- net LED: track 76.2 -> 0.00 mm, vias 1 -> 0
- net d1: track 0.00 -> 76.2 mm
- net d10: track 0.00 -> 74.1 mm, vias 0 -> 1
- net d2: track 0.00 -> 67.9 mm
- net d9: track 0.00 -> 65.8 mm, vias 0 -> 1
- net Net-(C1-Pad1): track 0.00 -> 63.2 mm
- net d3: track 0.00 -> 59.6 mm
- net d8: track 0.00 -> 57.7 mm, vias 0 -> 1
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Other:
- outline, holes or cut-outs redrawn
- board text added: "C"
- board text added: "D"
- board text added: "G"
- board text added: "OFF"
- board text added: "ON"
- board text added: "V"
