File: palmrest/palmrest.kicad_pcb (KiCad board)
At the start: 2 copper layers, 86 x 48.1 mm, 17 parts, among them J1 MJ-4PP-9, J2 Conn_01x05_Female, J3 Conn_01x10_Female, J4 Conn_01x05_Female, SW1 SW_SPDT, U1 XIAO, U2 XIAO, U3 HT7733A

Commit message: revenge 4
Parts:
- removed the G*** at (166.6, 96.2) (x2)
- removed the J3 at (158.2, 84.8)
- added G***: LOGO, mammoth:mammoth, F.Cu at (182.5, 78.8)
- added G***: LOGO, mammoth:mammoth, B.Cu at (182.5, 78.8)
- moved U3 75.3 mm to (126.0, 85.6)
- moved D1 51.5 mm to (124.7, 92.0), turned to -90 degrees
- moved C2 46.4 mm to (136.2, 90.7), turned to 180 degrees
- moved C1 34.8 mm to (136.2, 81.3), turned to 180 degrees
- moved U1 13.6 mm to (162.2, 79.2)
- moved U2 13.6 mm to (144.4, 79.2)
- moved R1 5.96 mm to (198.0, 93.1)
- moved R2 4.96 mm to (192.9, 93.1)
- moved SW1 0.98 mm to (178.2, 96.6)
- moved L1 0.37 mm to (126.7, 74.0)
- renumbered J4 to J3
Connections:
- J1 pad B: SCL -> VDD
- J1 pad D: VDD -> SCL
Routing:
- net SDA: track 192.5 -> 125.4 mm, vias 0 -> 1
- net GND: track 278.8 -> 215.8 mm, vias 7 -> 4
- net Net-(L1-Pad2): track 80.1 -> 27.6 mm
- net d10: track 74.1 -> 45.9 mm
- net VDD: track 209.8 -> 183.3 mm, vias 0 -> 1
- net INT: track 82.4 -> 56.1 mm, vias 1 -> 2
- net d9: track 65.8 -> 39.8 mm
- net VCC: track 95.0 -> 69.7 mm, vias 1 -> 3
- net d8: track 57.7 -> 32.5 mm
- net SCL: track 133.7 -> 109.2 mm
- net d7: track 33.2 -> 22.7 mm
- net Net-(C1-Pad1): track 63.2 -> 68.1 mm
- net d1: track 76.2 -> 71.8 mm, vias 0 -> 1
- net d2: track 67.9 -> 64.1 mm, vias 0 -> 1
- net d0: track 85.6 -> 81.9 mm, vias 0 -> 1
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Other:
- outline, holes or cut-outs redrawn
- board text added: "STEP 2 REVENGE 4"
