File: palmrest/palmrest.kicad_sch (KiCad schematic)
At the start: 15 parts, among them J2 Conn_01x05_Female, J3 Conn_01x05_Female, J4 Conn_01x12_Female, J5 Conn_01x12_Female, SW2 SW_SPDT

Commit message: revenge3
Parts:
- removed BT1, BT2: Battery_Cell, mammoth:ch28-2032LF_rev, symbol Device:Battery_Cell
- removed C1: C, mammoth:C_1206_3216Metric_Pad1.33x1.80mm_HandSolder_rev, symbol Device:C
- removed D1, D2: D, mammoth:D_SOD-323_HandSoldering_rev, symbol Device:D
- removed J3: Conn_01x05_Female, mammoth:JST_ACH_BM05B-ACHSS-A-GAN-ETF_1x05-1MP_P1.20mm_Vertical, symbol Connector:Conn_01x05_Female
- removed J4, J5: Conn_01x12_Female, mammoth:PinHeader_1x12_P2.54mm_Vertical, symbol Connector:Conn_01x12_Female
- removed SW1: (no value), symbol mammoth:SW_PUSH
- removed SW2: SW_SPDT, mammoth:SS-12D00G3, symbol Switch:SW_SPDT
- removed U1: (no value), symbol mammoth:ProMicro
- added BT1: Battery_Cell, mammoth:bat_case_AAA, symbol mammoth:Battery_Cell
- added C1: 47μF, mammoth:CP_Radial_D5.0mm_P2.00mm_P5.00mm_rev, symbol Device:C_Polarized
- added C2: 22μF, mammoth:CP_Radial_D5.0mm_P2.00mm_P5.00mm_rev, symbol Device:C_Polarized
- added D1: D_Schottky, symbol Device:D_Schottky
- added J3: Conn_01x10_Female, Connector_PinHeader_2.54mm:PinHeader_2x05_P2.54mm_Vertical, symbol Connector:Conn_01x10_Female
- added J4: Conn_01x05_Female, Connector_PinHeader_2.54mm:PinHeader_1x05_P2.54mm_Vertical, symbol Connector:Conn_01x05_Female
- added L1: 100μH, symbol Device:L
- added SW1: SW_SPDT, mammoth:SS-12D00G3, symbol Switch:SW_SPDT
- added U1, U2: XIAO, mammoth:Seeeduino XIAO-MOUDLE14P-2.54-21X17.8MM, symbol mammoth:XIAO
- added U3: HT7733A, mammoth:HT7733A, symbol mammoth:HT7733A
- J1: value (none) -> MJ-4PP-9; footprint (none) -> mammoth:MJ-4PP-9
- J2: footprint mammoth:JST_ACH_BM05B-ACHSS-A-GAN-ETF_1x05-1MP_P1.20mm_Vertical -> mammoth:JST_ACH_BM05B-ACHSS-A-GAN-ETF_1x05-1MP_P1.20mm_Vertical_rev
Connections:
- net GND: now also J1.A, BT1.2 (-), C1.2, C2.2, J3.10 (Pin_10), J4.4 (Pin_4), U1.13 (GND), U2.13 (GND), U3.1 (GND); no longer J1.C
- net SCL: now also J4.5 (Pin_5), U1.6 (PA9_A5_D5_SCL), U2.6 (PA9_A5_D5_SCL)
- net SDA: now also J1.C, J4.2 (Pin_2), U1.5 (PA8_A4_D4_SDA), U2.5 (PA8_A4_D4_SDA); no longer J1.A
- net VCC: now also U1.14 (5V), U2.14 (5V); no longer J1.D, J2.3 (Pin_3), R1.1, R2.1
- net LED renamed INT
- net INT: now also J4.1 (Pin_1), U1.7 (PB08_A6_D6_TX), U2.7 (PB08_A6_D6_TX)
- new net: C1.1, L1.1, SW1.1 (A)
- new net: D1.2 (A), L1.2, U3.3 (IN)
- new net: BT1.1 (+), SW1.2 (B)
- new net VDD: C2.1, D1.1 (K), J1.D, J2.3 (Pin_3), J3.9 (Pin_9), J4.3 (Pin_3), R1.1, R2.1, U1.12 (3V3), U2.12 (3V3), U3.2 (OUT)
- new net d0: J3.8 (Pin_8), U1.1 (PA02_A0_D0), U2.1 (PA02_A0_D0)
- new net d1: J3.6 (Pin_6), U1.2 (PA4_A1_D1), U2.2 (PA4_A1_D1)
- new net d10: J3.7 (Pin_7), U1.11 (PA6_A10_D10_MOSI), U2.11 (PA6_A10_D10_MOSI)
- new net d2: J3.4 (Pin_4), U1.3 (PA10_A2_D2), U2.3 (PA10_A2_D2)
- new net d3: J3.2 (Pin_2), U1.4 (PA11_A3_D3), U2.4 (PA11_A3_D3)
- new net d7: J3.1 (Pin_1), U1.8 (PB09_A7_D7_RX), U2.8 (PB09_A7_D7_RX)
- new net d8: J3.3 (Pin_3), U1.9 (PA7_A8_D8_SCK), U2.9 (PA7_A8_D8_SCK)
- new net d9: J3.5 (Pin_5), U1.10 (PA5_A9_D9_MISO), U2.10 (PA5_A9_D9_MISO)
Other:
- moved on the sheet: J1, J2

Commit message: revenge 4
Parts:
- removed J3: Conn_01x10_Female, Connector_PinHeader_2.54mm:PinHeader_2x05_P2.54mm_Vertical, symbol Connector:Conn_01x10_Female
- D1: footprint (none) -> mammoth:D_DO-34_SOD68_P7.62mm_Horizontal
- J3: renamed from J4; value Conn_01x05_Female -> (none); footprint Connector_PinHeader_2.54mm:PinHeader_1x05_P2.54mm_Vertical -> (none)
- L1: footprint (none) -> mammoth:L_Radial_D10.0mm_P5.00mm_Fastron_07M
Connections:
- net SCL: now also J1.D; no longer J1.B
- net VDD: now also J1.B; no longer J1.D
